File: circuits/controller/access-controller.kicad_sch (KiCad schematic)
At the start: 68 parts, among them J1 Conn_01x01_Female, J10 Terminal_01x03, J11 Terminal_01x04, J12 Screw_Terminal_01x05, J13 Conn_02x06_Odd_Even, J14 Terminal_01x04, J15 Terminal_01x03, J16 Terminal_01x03, J17 Terminal_01x03, J18 Terminal_01x04, J19 Screw_Terminal_01x05, J2 Conn_01x01_Female, J22 RF_MODULE, J3 Conn_01x01_Female, J4 Conn_01x01_Female, J6 Screw_Terminal_01x02, J7 Terminal_01x04, J8 Terminal_01x03, J9 Barrel_Jack_Switch, J9 Terminal_01x03, Q3 Q_MMBT5551, Q4 Q_MMBT5551, U1 MCP23017_SS

Commit message: fix(hardware): correct Wiegand input biasing
Parts:
- removed D24, D26, D29, D30: White, LED_SMD:LED_0603_1608Metric_Pad1.05x0.95mm_HandSolder, symbol open_automation:LED-0603-W
- R35, R74, R77, R78: value 10K -> 4.7K; LCSC C25744 -> C25900; Part Number 0402WGF1002TCE -> 0402WGF4701TCE
Connections:
- net 5V: now also R35.2, R74.2, R77.2, R78.2
- net GND: no longer R35.1, R74.1, R77.1, R78.1
- net WG0_DATA0: now also R74.1
- net WG0_DATA1: now also R78.1
- net WG1_DATA0: now also R35.1
- net WG1_DATA1: now also R77.1
Other:
- moved on the sheet: R35, R74, R77, R78

Commit message: chore(hardware): upgrade KiCad project to Eeschema 10.0 format
Re-saved in KiCad 10 (generator_version bump, new zone-fill and
footprint-default schema fields, float precision cleanup). Verified
component counts (lib_id) are unchanged in every schematic sheet -
formatting only, no circuit edits.
Parts:
- renumbered J9 to J5
