File: circuits/controller/microcontroller.kicad_sch (KiCad schematic)
At the start: 35 parts, among them J8 USB_MINI_B, J9 USB_MINI_B, Q1 Q_L8050QLT1G, Q2 Q_L8550HQLT1G, U1 CP2102N-Axx-xQFN28, U3 ESP32-S3-WROOM-1

Commit message: chore(hardware): upgrade KiCad project to Eeschema 10.0 format
Re-saved in KiCad 10 (generator_version bump, new zone-fill and
footprint-default schema fields, float precision cleanup). Verified
component counts (lib_id) are unchanged in every schematic sheet -
formatting only, no circuit edits.
Parts:
- renumbered C40 to C10, C41 to C11, C43 to C12, C44 to C13, C48 to C14, C42 to C15, C47 to C9, D13 to D10, D17 to D11, D14 to D5, D11 to D6, D15 to D7, D16 to D8, D10 to D9, J9 to J20, J8 to J21, R39 to R20, R40 to R21, R34 to R22, R33 to R23, R32 to R24, R35 to R25, R36 to R26, R37 to R27, R38 to R28, R30 to R29, R31 to R30, U1 to U6, U3 to U7
