File: circuits/controller/power.kicad_sch (KiCad schematic)
At the start: 19 parts, among them U3 REG_AMS1117-3.3, U4 MIC29302WU, U4 REG_MT2492

Commit message: chore(hardware): upgrade KiCad project to Eeschema 10.0 format
Re-saved in KiCad 10 (generator_version bump, new zone-fill and
footprint-default schema fields, float precision cleanup). Verified
component counts (lib_id) are unchanged in every schematic sheet -
formatting only, no circuit edits.
Parts:
- renumbered C33 to C16, C36 to C17, C37 to C18, L7 to L1, R11 to R6, R12 to R7, U4 to U8
